Commit message: колёса не работают

File: models/diff_drive_robot/urdf/diff_drive_robot.xacro (robot description, xacro)
@@ -1,6 +1,9 @@
 <?xml version='1.0'?>
 <robot name="robot" xmlns:xacro="http://www.ros.org/wiki/xacro">
-  <xacro:include filename="$(find roscourse_2023_project_scene)/models/diff_drive_robot/urdf/diff_drive_robot.gazebo" />
-  <xacro:include filename="$(find roscourse_2023_project_scene)/models/diff_drive_robot/urdf/materials.xacro" />
+  <xacro:property name="pack" value="roscourse_2023_project_scene" />
+  <xacro:include filename="$(find ${pack})/models/diff_drive_robot/urdf/diff_drive_robot.gazebo" />
+  <xacro:include filename="$(find ${pack})/models/diff_drive_robot/urdf/materials.xacro" />
+  <xacro:include filename="$(find ${pack})/models/diff_drive_robot/urdf/inertial.urdf.xacro" />
+  <xacro:include filename="$(find ${pack})/models/diff_drive_robot/urdf/wheel.xacro" />
   <link name='base'>
     <pose>0 0 0.0 0 0 0</pose>
@@ -19,11 +22,11 @@
       </geometry>
     </collision>
-    <visual name='base_visual'>
-      <origin xyz="0 0 0" rpy=" 0 0 0"/>
-      <geometry>
-        <box size=".6 .4 .2"/>
-      </geometry>
-      <material name="orange"/>
-    </visual>
+  <visual name='base_visual'>
+    <origin xyz="0 0 -0.1" rpy=" 0 0 0"/>
+    <geometry>
+      <mesh filename="$(find roscourse_2023_project_scene)/models/Subaru.stl" scale="0.25 0.25 0.25"/>
+    </geometry>
+    <material name="blue"/>
+  </visual>
     <collision name='caster_collision_rear'>
       <origin xyz="-0.24 0 -0.08" rpy=" 0 0 0"/>
@@ -73,77 +76,8 @@
     </visual>
   </link>
-  <link name="left_wheel">
-    <collision name="collision">
-      <origin xyz="0 0 0" rpy="0 1.5707 1.5707"/>
-      <geometry>
-        <cylinder radius="0.1" length="0.05"/>
-      </geometry>
-    </collision>
-    <visual name="left_wheel_visual">
-      <origin xyz="0 0 0" rpy="0 1.5707 1.5707"/>
-      <geometry>
-        <cylinder radius="0.1" length="0.05"/>
-      </geometry>
-      <material name="green"/>
-    </visual>
-    <inertial>
-      <origin xyz="0 0 0" rpy="0 1.5707 1.5707"/>
-      <mass value="5"/>
-      <cylinder_inertia m="5" r="0.1" h="0.05"/>
-      <inertia
-        ixx="1.0" ixy="0.0" ixz="0.0"
-        iyy="1.0" iyz="0.0"
-        izz="1.0"/>
-    </inertial>
-  </link>
-  <link name="right_wheel">
-    <collision name="collision">
-      <origin xyz="0 0 0" rpy="0 1.5707 1.5707"/>
-      <geometry>
-        <cylinder radius="0.1" length="0.05"/>
-      </geometry>
-    </collision>
-    <visual name="right_wheel_visual">
-      <origin xyz="0 0 0" rpy="0 1.5707 1.5707"/>
-      <geometry>
-        <cylinder radius="0.1" length="0.05"/>
-      </geometry>
-      <material name="green"/>
-    </visual>
-    <inertial>
-      <origin xyz="0 0 0" rpy="0 1.5707 1.5707"/>
-      <mass value="5"/>
-      <cylinder_inertia m="5" r="0.1" h="0.05"/>
-      <inertia
-        ixx="1.0" ixy="0.0" ixz="0.0"
-        iyy="1.0" iyz="0.0"
-        izz="1.0"/>
-    </inertial>
-  </link>
-  <link name='camera2'>
-    <visual name='camera_visual'>
-      <origin xyz="0 0 0" rpy=" 0 0 0"/>
-      <geometry>
-        <box size=".05 .05 .05"/>
-      </geometry>
-      <material name="white"/>
-    </visual>
-  </link>
-  <joint type="continuous" name="left_wheel_hinge">
-    <origin xyz="0.05 0.226 -0.05" rpy="0 0 0"/>
-    <child link="left_wheel"/>
-    <parent link="base"/>
-    <axis xyz="0 1 0" rpy="0 0 0"/>
-    <limit effort="100" velocity="100"/>
-    <joint_properties damping="0.0" friction="0.0"/>
-  </joint>
-  <joint type="continuous" name="right_wheel_hinge">
-    <origin xyz="0.05 -0.226 -0.05" rpy="0 0 0"/>
-    <child link="right_wheel"/>
-    <parent link="base"/>
-    <axis xyz="0 1 0" rpy="0 0 0"/>
-    <limit effort="100" velocity="100"/>
-    <joint_properties damping="0.0" friction="0.0"/>
-  </joint>
+  <xacro:wheel side="up_left" x="0.1" y="0.09" z="0.0" sign="1"/>
+  <xacro:wheel side="up_right" x="0.1" y="0.09" z="0.0" sign="-1"/>
+  <xacro:wheel side="down_left" x="0.1" y="-0.09" z="0.0" sign="1"/>
+  <xacro:wheel side="down_right" x="0.1" y="-0.09" z="0.0" sign="-1"/>
   <joint type="fixed" name="camera_joint">
     <origin xyz="0.3 0 0" rpy="0 0 0"/>

Commit message: rviz?

File: models/diff_drive_robot/urdf/diff_drive_robot.xacro (robot description, xacro)
@@ -80,8 +80,3 @@
   <xacro:wheel side="down_left" x="0.1" y="-0.09" z="0.0" sign="1"/>
   <xacro:wheel side="down_right" x="0.1" y="-0.09" z="0.0" sign="-1"/>
-  <joint type="fixed" name="camera_joint">
-    <origin xyz="0.3 0 0" rpy="0 0 0"/>
-    <child link="camera2"/>
-    <parent link="base"/>
-  </joint>
 </robot>

File: models/diff_drive_robot/urdf/wheel.xacro (robot description, xacro)
@@ -26,5 +26,5 @@
             <joint_properties damping="0.5" friction="0.1"/>
             <child link="wheel_${side}_link"/>
-            <parent link="base_link"/>
+            <parent link="base"/>
         </joint>
         <transmission name="wheel_${side}_trans">

Commit message: pack

File: models/diff_drive_robot/urdf/diff_drive_robot.xacro (robot description, xacro)
@@ -1,82 +1,67 @@
 <?xml version='1.0'?>
-<robot name="robot" xmlns:xacro="http://www.ros.org/wiki/xacro">
-  <xacro:property name="pack" value="roscourse_2023_project_scene" />
-  <xacro:include filename="$(find ${pack})/models/diff_drive_robot/urdf/diff_drive_robot.gazebo" />
-  <xacro:include filename="$(find ${pack})/models/diff_drive_robot/urdf/materials.xacro" />
-  <xacro:include filename="$(find ${pack})/models/diff_drive_robot/urdf/inertial.urdf.xacro" />
-  <xacro:include filename="$(find ${pack})/models/diff_drive_robot/urdf/wheel.xacro" />
-  <link name='base'>
-    <pose>0 0 0.0 0 0 0</pose>
-    <inertial>
-      <mass value="20.0"/>
-      <origin xyz="0.0 0 0.1" rpy=" 0 0 0"/>
-      <inertia
-          ixx="0.5" ixy="0" ixz="0"
-          iyy="1.0" iyz="0"
-          izz="0.1"
-      />
-    </inertial>
-    <collision name='collision'>
-      <geometry>
-        <box size=".6 .4 .2"/>
-      </geometry>
-    </collision>
-  <visual name='base_visual'>
-    <origin xyz="0 0 -0.1" rpy=" 0 0 0"/>
-    <geometry>
-      <mesh filename="$(find roscourse_2023_project_scene)/models/Subaru.stl" scale="0.25 0.25 0.25"/>
-    </geometry>
-    <material name="blue"/>
-  </visual>
-    <collision name='caster_collision_rear'>
-      <origin xyz="-0.24 0 -0.08" rpy=" 0 0 0"/>
-      <geometry>
-        <sphere radius="0.06"/>
-      </geometry>
-      <surface>
-        <friction>
-          <ode>
-            <mu>0</mu>
-            <mu2>0</mu2>
-            <slip1>1.0</slip1>
-            <slip2>1.0</slip2>
-          </ode>
-        </friction>
-      </surface>
-    </collision>
-    <visual name='caster_visual_rear'>
-      <origin xyz="-0.24 0 -0.08" rpy=" 0 0 0"/>
-      <geometry>
-        <sphere radius="0.06"/>
-      </geometry>
-      <material name="white"/>
-    </visual>
-    <collision name='caster_collision_forward'>
-      <origin xyz="0.24 0 -0.08" rpy=" 0 0 0"/>
-      <geometry>
-        <sphere radius="0.06"/>
-      </geometry>
-      <surface>
-        <friction>
-          <ode>
-            <mu>0</mu>
-            <mu2>0</mu2>
-            <slip1>1.0</slip1>
-            <slip2>1.0</slip2>
-          </ode>
-        </friction>
-      </surface>
-    </collision>
-    <visual name='caster_visual_forward'>
-      <origin xyz="0.24 0 -0.08" rpy=" 0 0 0"/>
-      <geometry>
-        <sphere radius="0.06"/>
-      </geometry>
-      <material name="white"/>
-    </visual>
-  </link>
-  <xacro:wheel side="up_left" x="0.1" y="0.09" z="0.0" sign="1"/>
-  <xacro:wheel side="up_right" x="0.1" y="0.09" z="0.0" sign="-1"/>
-  <xacro:wheel side="down_left" x="0.1" y="-0.09" z="0.0" sign="1"/>
-  <xacro:wheel side="down_right" x="0.1" y="-0.09" z="0.0" sign="-1"/>
+<robot name="cart_robot" xmlns:xacro="http://www.ros.org/wiki/xacro" >
+<xacro:property name="side" value="right"/>
+<xacro:property name="pack" value="my_robot_simulation_control" />
+<xacro:include filename="$(find ${pack})/urdf/materials.xacro" />
+<xacro:include filename="$(find ${pack})/urdf/wheel.xacro" />
+<xacro:include filename="$(find ${pack})/urdf/inertial.urdf.xacro" />
+<xacro:include filename="$(find ${pack})/urdf/setup.gazebo" />
+<!-- robot_arm BUT NOW cart_robot -->
+<origin xyz="0.0 0.0 0.0" rpy="0.0 0.0 0.0"/>
+    <link name="base_footprint"/>
+    <joint name="base_joint" type="fixed">
+        <origin rpy="0 0 0" xyz="0 0 0.0102"/>
+        <parent link="base_footprint"/>
+        <child link="base_link"/>
+    </joint>
+    <link name='base_link'>
+        <visual name='base_visual'>
+        <origin xyz="0.0 0.0 0.0" rpy="0.0 0.0 0.0"/>
+        <geometry>
+        <box size="0.2 0.18 0.12 "/>
+        </geometry>
+        <material name="blue"/>
+        </visual>
+        <xacro:inertial_box mass="2" x="0.2" y="0.18" z="0.12" >
+            <origin xyz="0.0 0.0 0.0" rpy="0.0 0.0 0.0"/>
+        </xacro:inertial_box>
+        <collision>
+            <origin xyz="0.0 0.0 0.0" rpy="0.0 0.0 0.0"/>
+                <geometry>
+                    <box size="0.2 0.18 0.12 "/>
+                </geometry>
+        </collision>
+    </link>
+    <link name='camera'>
+        <visual name='camera_visual'>
+        <origin xyz="0 0 0" rpy=" 0 0 1.570796"/>
+        <geometry>
+            <box size=".05 .05 .05"/>
+        </geometry>
+        <material name="gray"/>
+        </visual>
+    </link>
+    <joint type="fixed" name="camera_joint">
+        <origin xyz="0 0.10 0.10" rpy="0 0 1.570796"/>
+        <child link="camera"/>
+        <parent link="base_link"/>
+    </joint>
+    <link name="lidar">
+        <visual name='lidar_visual'>
+            <origin xyz="0 0 0" rpy=" 0 0 0"/>
+            <geometry>
+                <box size=".05 .05 .05"/>
+            </geometry>
+            <material name="red"/>
+        </visual>
+    </link>
+    <joint name="lidar_joint" type="fixed">
+        <origin xyz="0 0.10 0.20" rpy="0 0 1.570796"/>
+        <child link="lidar"/>
+        <parent link="base_link"/>
+    </joint>
+    <xacro:wheel side="up_left" x="0.1" y="0.09" z="0.0" sign="1"/>
+    <xacro:wheel side="up_right" x="0.1" y="0.09" z="0.0" sign="-1"/>
+    <xacro:wheel side="down_left" x="0.1" y="-0.09" z="0.0" sign="1"/>
+    <xacro:wheel side="down_right" x="0.1" y="-0.09" z="0.0" sign="-1"/>
 </robot>
