Commit message: pack менять теперь только один раз

File: models/project_robot/urdf/diff_drive_robot.xacro (robot description, xacro)
@@ -1,6 +1,11 @@
 <?xml version='1.0'?>
 <robot name="robot" xmlns:xacro="http://www.ros.org/wiki/xacro">
-  <xacro:include filename="$(find roscourse_2023_project_scene)/models/diff_drive_robot/urdf/diff_drive_robot.gazebo" />
-  <xacro:include filename="$(find roscourse_2023_project_scene)/models/diff_drive_robot/urdf/materials.xacro" />
+  <xacro:property name="pack" value="roscourse_2023_project_scene" />
+  <!-- <xacro:include filename="$(find ${pack})/urdf/materials.xacro" />
+  <xacro:include filename="$(find ${pack})/urdf/wheel.xacro" />
+  <xacro:include filename="$(find ${pack})/urdf/inertial.urdf.xacro" />
+  <xacro:include filename="$(find ${pack})/urdf/setup.gazebo" /> -->
+  <xacro:include filename="$(find ${pack})/models/diff_drive_robot/urdf/diff_drive_robot.gazebo" />
+  <xacro:include filename="$(find ${pack})/models/diff_drive_robot/urdf/materials.xacro" />
   <link name='base'>
     <pose>0 0 0.0 0 0 0</pose>
