Commit message: added robot model

File: models/project_robot/urdf/materials.xacro (robot description, xacro)
@@ -3,4 +3,7 @@
   <material name="black">
     <color rgba="0.0 0.0 0.0 1.0"/>
+  </material>
+  <material name="white">
+    <color rgba="1.0 1.0 1.0 1.0"/>
   </material>
   <material name="blue">
@@ -25,3 +28,12 @@
     <color rgba="1.0 1.0 1.0 1.0"/>
   </material>
+    <material name="gold">
+        <color rgba="0.5 0.3 0.6 1.0"/>
+    </material>
+    <material name="another1">
+        <color rgba="0.15 0.2 0.8 1.0"/>
+    </material>
+    <material name="another2">
+        <color rgba="0.7 0.25 0.1 1.0"/>
+    </material>
 </robot>

Commit message: fixes

File: models/project_robot/urdf/materials.xacro (robot description, xacro)
@@ -3,7 +3,4 @@
   <material name="black">
     <color rgba="0.0 0.0 0.0 1.0"/>
-  </material>
-  <material name="white">
-    <color rgba="1.0 1.0 1.0 1.0"/>
   </material>
   <material name="blue">

File: models/project_robot/urdf/robot_model.xacro (robot description, xacro)
@@ -1,9 +1,9 @@
 <?xml version='1.0'?>
-<robot name="cart_robot" xmlns:xacro="http://www.ros.org/wiki/xacro" >
+<robot name="project_robot" xmlns:xacro="http://www.ros.org/wiki/xacro" >
 <xacro:property name="side" value="right"/>
-<xacro:include filename="$(find my_robot_simulation_control)/urdf/materials.xacro" />
-<xacro:include filename="$(find my_robot_simulation_control)/urdf/wheel.xacro" />
-<xacro:include filename="$(find my_robot_simulation_control)/urdf/inertial.urdf.xacro" />
-<xacro:include filename="$(find my_robot_simulation_control)/urdf/setup.gazebo" />
+<xacro:include filename="$(find roscourse_2023_project_scene)/models/project_robot/urdf/materials.xacro" />
+<xacro:include filename="$(find roscourse_2023_project_scene)/models/project_robot/urdf/wheel.xacro" />
+<xacro:include filename="$(find roscourse_2023_project_scene)/models/project_robot/urdf/inertial.urdf.xacro" />
+<xacro:include filename="$(find roscourse_2023_project_scene)/models/project_robot/urdf/setup.gazebo" />
 <!-- robot_arm BUT NOW cart_robot -->
 <origin xyz="0.0 0.0 0.0" rpy="0.0 0.0 0.0"/>

Commit message: fixes

File: models/project_robot/urdf/materials.xacro (robot description, xacro)
@@ -25,12 +25,3 @@
     <color rgba="1.0 1.0 1.0 1.0"/>
   </material>
-    <material name="gold">
-        <color rgba="0.5 0.3 0.6 1.0"/>
-    </material>
-    <material name="another1">
-        <color rgba="0.15 0.2 0.8 1.0"/>
-    </material>
-    <material name="another2">
-        <color rgba="0.7 0.25 0.1 1.0"/>
-    </material>
 </robot>

File: models/project_robot/urdf/robot_model.xacro (robot description, xacro)
@@ -1,14 +1,12 @@
 <?xml version='1.0'?>
 <robot name="project_robot" xmlns:xacro="http://www.ros.org/wiki/xacro" >
-<xacro:property name="side" value="right"/>
 <xacro:include filename="$(find roscourse_2023_project_scene)/models/project_robot/urdf/materials.xacro" />
-<xacro:include filename="$(find roscourse_2023_project_scene)/models/project_robot/urdf/wheel.xacro" />
 <xacro:include filename="$(find roscourse_2023_project_scene)/models/project_robot/urdf/inertial.urdf.xacro" />
 <xacro:include filename="$(find roscourse_2023_project_scene)/models/project_robot/urdf/setup.gazebo" />
-<!-- robot_arm BUT NOW cart_robot -->
+<xacro:include filename="$(find roscourse_2023_project_scene)/models/project_robot/urdf/wheel.xacro" />
 <origin xyz="0.0 0.0 0.0" rpy="0.0 0.0 0.0"/>
     <link name="base_footprint"/>
     <joint name="base_joint" type="fixed">
-        <origin rpy="0 0 0" xyz="0 0 0.0102"/>
+        <origin rpy="0 0 0" xyz="0 0 0"/>
         <parent link="base_footprint"/>
         <child link="base_link"/>
@@ -17,8 +15,8 @@
         <visual name='base_visual'>
         <origin xyz="0.0 0.0 0.0" rpy="0.0 0.0 0.0"/>
-        <geometry>
-        <box size="0.2 0.18 0.12 "/>
-        </geometry>
-        <material name="blue"/>
+            <geometry>
+                <box size="0.2 0.18 0.12 "/>
+            </geometry>
+            <material name="black"/>
         </visual>
         <xacro:inertial_box mass="2" x="0.2" y="0.18" z="0.12" >
@@ -38,9 +36,9 @@
                 <box size=".05 .05 .05"/>
             </geometry>
-            <material name="red"/>
+            <material name="black"/>
         </visual>
     </link>
     <joint name="lidar_joint" type="fixed">
-        <origin xyz="0 0.10 0.20" rpy="0 0 1.570796"/>
+        <origin xyz="0 0.10 0.20" rpy="0 0 ${pi/2}"/>
         <child link="lidar"/>
         <parent link="base_link"/>

File: models/project_robot/urdf/wheel.xacro (robot description, xacro)
@@ -4,15 +4,15 @@
         <link name='wheel_${side}_link'>
             <visual name='wheel_${side}_visual'>
-            <origin xyz="${(sign*0.1)/8} 0 0" rpy="0 1.57 0"/>
+                <origin xyz="${(sign*0.1)/8} 0 0" rpy="0 ${pi/2} 0"/>
                 <geometry>
                     <cylinder length="${(0.1)/4}" radius="${0.15/2}"/>
                 </geometry>
-                <material name="red"/>
+                <material name="orange"/>
             </visual>
-            <xacro:inertial_cylinder mass="5" length="0.5" radius="0.25">
-                <origin xyz="${(sign*0.1)/8} 0 0" rpy="0 1.57 0"/>
+            <xacro:inertial_cylinder mass="5" length="${(0.1)/4}" radius="${0.15/2}">
+                <origin xyz="${(sign*0.1)/8} 0 0" rpy="0 ${pi/2} 0"/>
             </xacro:inertial_cylinder>
             <collision>
-               <origin xyz="${(sign*0.1)/8} 0 0" rpy="0 1.57 0"/>
+               <origin xyz="${(sign*0.1)/8} 0 0" rpy="0 ${pi/2} 0"/>
                 <geometry>
                     <cylinder length="${(0.1)/4}" radius="${0.15/2}"/>
