Commit message: another fixes

File: models/project_robot/urdf/inertial.urdf.xacro (robot description, xacro)
@@ -1,10 +1,4 @@
 <?xml version="1.0"?>
 <robot xmlns:xacro="http://www.ros.org/wiki/xacro">
-<!--
-    EXAMPLE OF USE IN EXTERNAL FILE
-<xacro:inertial_box mass="0.5" x="0.5" y="0.25" z="0.15">
-            <origin xyz="0 0 0.075" rpy="0 0 0"/>
-        </xacro:inertial_box>
-         -->
     <xacro:macro name="inertial_sphere" params="mass radius *origin">
         <inertial>

File: models/project_robot/urdf/robot_model.xacro (robot description, xacro)
@@ -11,7 +11,7 @@
         <origin rpy="0 0 0" xyz="0 0 0"/>
         <parent link="base_footprint"/>
-        <child link="base_link"/>
+        <child link="base"/>
     </joint>
-    <link name='base_link'>
+    <link name='base'>
         <visual name='base_visual'>
         <origin xyz="0.0 0.0 0.0" rpy="0.0 0.0 0.0"/>
@@ -19,5 +19,5 @@
                 <box size="0.2 0.18 0.12 "/>
             </geometry>
-            <material name="black"/>
+            <material name="orange"/>
         </visual>
         <xacro:inertial_box mass="10" x="0.2" y="0.18" z="0.12" >
@@ -37,11 +37,11 @@
                 <box size=".05 .05 .05"/>
             </geometry>
-            <material name="black"/>
+            <material name="red"/>
         </visual>
     </link>
     <joint name="lidar_joint" type="fixed">
-        <origin xyz="0 0.10 0.20" rpy="0 0 ${pi/2}"/>
+        <origin xyz="0 0.10 0.08" rpy="0 0 ${pi/2}"/>
         <child link="lidar"/>
-        <parent link="base_link"/>
+        <parent link="base"/>
     </joint>
     <xacro:wheel side="up_left" x="0.1" y="0.09" z="0.0" sign="1"/>

File: models/project_robot/urdf/wheel.xacro (robot description, xacro)
@@ -8,5 +8,5 @@
                     <cylinder length="${(0.1)/4}" radius="${0.15/2}"/>
                 </geometry>
-                <material name="orange"/>
+                <material name="black"/>
             </visual>
             <xacro:inertial_cylinder mass="2.5" length="${(0.1)/4}" radius="${0.15/2}">
@@ -26,5 +26,5 @@
             <joint_properties damping="0.5" friction="0.1"/>
             <child link="wheel_${side}_link"/>
-            <parent link="base_link"/>
+            <parent link="base"/>
         </joint>
         <transmission name="wheel_${side}_trans">
