Commit message: fiiiixeees

File: models/project_robot/urdf/wheel.xacro (robot description, xacro)
@@ -2,5 +2,5 @@
 <robot xmlns:xacro="http://www.ros.org/wiki/xacro">
     <xacro:macro name="wheel" params="side x y z sign">
-        <link name='wheel_${side}_link'>
+        <link name='wheel_${side}'>
             <visual name='wheel_${side}_visual'>
                 <origin xyz="${(sign*0.1)/8} 0 0" rpy="0 ${pi/2} 0"/>
@@ -25,5 +25,5 @@
             <limit effort="100" velocity="50"/>
             <joint_properties damping="0.5" friction="0.1"/>
-            <child link="wheel_${side}_link"/>
+            <child link="wheel_${side}"/>
             <parent link="base"/>
         </joint>

Commit message: fd

File: models/project_robot/urdf/wheel.xacro (robot description, xacro)
@@ -17,5 +17,5 @@
                <origin xyz="${(sign*0.1)/8} 0 0" rpy="0 ${pi/2} 0"/>
                 <geometry>
-                    <cylinder length="${(0.1)/4}" radius="${0.17/2}"/>
+                    <cylinder length="${(0.1)/4}" radius="${0.15/2}"/>
                 </geometry>
             </collision>
