Commit message: init rotated robot, deleted camera

File: models/project_robot/urdf/robot_model.xacro (robot description, xacro)
@@ -32,18 +32,4 @@
         </collision>
     </link>
-    <link name='camera'>
-        <visual name='camera_visual'>
-        <origin xyz="0 0 0" rpy=" 0 0 1.570796"/>
-        <geometry>
-            <box size=".05 .05 .05"/>
-        </geometry>
-        <material name="red"/>
-        </visual>
-    </link>
-    <joint type="fixed" name="camera_joint">
-        <origin xyz="0 0.10 0.10" rpy="0 0 1.570796"/>
-        <child link="camera"/>
-        <parent link="base_link"/>
-    </joint>
     <link name="lidar">
         <visual name='lidar_visual'>

Commit message: changed physical properties of robot

File: models/project_robot/urdf/robot_model.xacro (robot description, xacro)
@@ -22,5 +22,5 @@
         <material name="blue"/>
         </visual>
-        <xacro:inertial_box mass="2" x="0.2" y="0.18" z="0.12" >
+        <xacro:inertial_box mass="10" x="0.2" y="0.18" z="0.12" >
             <origin xyz="0.0 0.0 0.0" rpy="0.0 0.0 0.0"/>
         </xacro:inertial_box>

File: models/project_robot/urdf/wheel.xacro (robot description, xacro)
@@ -10,5 +10,5 @@
                 <material name="red"/>
             </visual>
-            <xacro:inertial_cylinder mass="5" length="0.5" radius="0.25">
+            <xacro:inertial_cylinder mass="2.5" length="0.5" radius="0.25">
                 <origin xyz="${(sign*0.1)/8} 0 0" rpy="0 1.57 0"/>
             </xacro:inertial_cylinder>
@@ -23,5 +23,5 @@
             <origin xyz="${x*sign} ${y} ${z}" rpy="0 0 0"/>
             <axis xyz="1 0 0" />
-            <limit effort="50" velocity="100"/>
+            <limit effort="100" velocity="50"/>
             <joint_properties damping="0.5" friction="0.1"/>
             <child link="wheel_${side}_link"/>

Commit message: pack into robot

File: models/project_robot/urdf/robot_model.xacro (robot description, xacro)
@@ -1,9 +1,9 @@
 <?xml version='1.0'?>
 <robot name="project_robot" xmlns:xacro="http://www.ros.org/wiki/xacro" >
-<xacro:property name="side" value="right"/>
-<xacro:include filename="$(find roscourse_2023_project_scene)/models/project_robot/urdf/materials.xacro" />
-<xacro:include filename="$(find roscourse_2023_project_scene)/models/project_robot/urdf/wheel.xacro" />
-<xacro:include filename="$(find roscourse_2023_project_scene)/models/project_robot/urdf/inertial.urdf.xacro" />
-<xacro:include filename="$(find roscourse_2023_project_scene)/models/project_robot/urdf/setup.gazebo" />
+<xacro:property name="pack" value="roscourse_2023_project_scene" />
+<xacro:include filename="$(find ${pack})/models/project_robot/urdf/materials.xacro" />
+<xacro:include filename="$(find ${pack})/models/project_robot/urdf/wheel.xacro" />
+<xacro:include filename="$(find ${pack})/models/project_robot/urdf/inertial.urdf.xacro" />
+<xacro:include filename="$(find ${pack})/models/project_robot/urdf/setup.gazebo" />
 <!-- robot_arm BUT NOW cart_robot -->
 <origin xyz="0.0 0.0 0.0" rpy="0.0 0.0 0.0"/>

Commit message: Vizual and ISU ID

File: models/project_robot/urdf/robot_model.xacro (robot description, xacro)
@@ -15,9 +15,9 @@
     <link name='base'>
         <visual name='base_visual'>
-        <origin xyz="0.0 0.0 0.0" rpy="0.0 0.0 0.0"/>
+            <origin xyz="0.033 -0.025 -0.05" rpy=" 0 0 ${-pi/2}"/>
             <geometry>
-                <box size="0.2 0.18 0.12 "/>
+            <mesh filename="$(find ${pack})/models/Subaru_Impreza.stl" scale="0.08 0.1 0.11"/>
             </geometry>
-            <material name="orange"/>
+                <material name="orange"/>
         </visual>
         <xacro:inertial_box mass="10" x="0.2" y="0.18" z="0.12" >
@@ -27,5 +27,5 @@
             <origin xyz="0.0 0.0 0.0" rpy="0.0 0.0 0.0"/>
                 <geometry>
-                    <box size="0.2 0.18 0.12 "/>
+                    <box size="0.2 0.36 0.12 "/>
                 </geometry>
         </collision>
@@ -35,5 +35,5 @@
             <origin xyz="0 0 0" rpy=" 0 0 0"/>
             <geometry>
-                <box size=".05 .05 .05"/>
+                <box size=".025 .025 .025"/>
             </geometry>
             <material name="red"/>
@@ -41,11 +41,11 @@
     </link>
     <joint name="lidar_joint" type="fixed">
-        <origin xyz="0 0.10 0.08" rpy="0 0 ${pi/2}"/>
+        <origin xyz="0 0.15 0.0" rpy="0 0 ${pi/2}"/>
         <child link="lidar"/>
         <parent link="base"/>
     </joint>
-    <xacro:wheel side="up_left" x="0.1" y="0.09" z="0.0" sign="1"/>
-    <xacro:wheel side="up_right" x="0.1" y="0.09" z="0.0" sign="-1"/>
-    <xacro:wheel side="down_left" x="0.1" y="-0.09" z="0.0" sign="1"/>
-    <xacro:wheel side="down_right" x="0.1" y="-0.09" z="0.0" sign="-1"/>
+    <xacro:wheel side="up_left" x="0.1" y="0.09" z="0.0" sign="1" sign2="2"/>
+    <xacro:wheel side="up_right" x="0.1" y="0.09" z="0.0" sign="-1" sign2="1"/>
+    <xacro:wheel side="down_left" x="0.1" y="-0.09" z="0.0" sign="1" sign2="2"/>
+    <xacro:wheel side="down_right" x="0.1" y="-0.09" z="0.0" sign="-1" sign2="1"/>
 </robot>

File: models/project_robot/urdf/wheel.xacro (robot description, xacro)
@@ -1,7 +1,15 @@
 <?xml version='1.0'?>
 <robot xmlns:xacro="http://www.ros.org/wiki/xacro">
-    <xacro:macro name="wheel" params="side x y z sign">
+    <xacro:macro name="wheel" params="side x y z sign sign2">
+        <xacro:property name="pack" value="roscourse_2023_project_scene" />
         <link name='wheel_${side}'>
             <visual name='wheel_${side}_visual'>
+            <origin xyz="${(sign*0.1)/8} 0 0" rpy="${sign2*pi} 0 ${pi/2}"/>
+            <geometry>
+            <mesh filename="$(find ${pack})/models/Wheel.stl" scale="0.0043 0.002 0.0043"/>
+            </geometry>
+                <material name="black"/>
+            </visual>
+            <!-- <visual name='wheel_${side}_visual'>
                 <origin xyz="${(sign*0.1)/8} 0 0" rpy="0 ${pi/2} 0"/>
                 <geometry>
@@ -9,6 +17,6 @@
                 </geometry>
                 <material name="black"/>
-            </visual>
-            <xacro:inertial_cylinder mass="2.5" length="${(0.1)/4}" radius="${0.15/2}">
+            </visual> -->
+            <xacro:inertial_cylinder mass="1" length="${(0.1)/4}" radius="${0.15/2}">
                 <origin xyz="${(sign*0.1)/8} 0 0" rpy="0 ${pi/2} 0"/>
             </xacro:inertial_cylinder>

Commit message: Better URDF

File: models/project_robot/urdf/robot_model.xacro (robot description, xacro)
@@ -7,25 +7,19 @@
 <xacro:include filename="$(find ${pack})/models/project_robot/urdf/setup.gazebo" />
 <origin xyz="0.0 0.0 0.0" rpy="0.0 0.0 0.0"/>
-    <link name="base_footprint"/>
-    <joint name="base_joint" type="fixed">
-        <origin rpy="0 0 0" xyz="0 0 0"/>
-        <parent link="base_footprint"/>
-        <child link="base"/>
-    </joint>
     <link name='base'>
         <visual name='base_visual'>
             <origin xyz="0.033 -0.025 -0.05" rpy=" 0 0 ${-pi/2}"/>
             <geometry>
-            <mesh filename="$(find ${pack})/models/Subaru_Impreza.stl" scale="0.08 0.1 0.11"/>
+                <mesh filename="$(find ${pack})/models/Subaru_Impreza.stl" scale="0.08 0.1 0.11"/>
             </geometry>
                 <material name="orange"/>
         </visual>
-        <xacro:inertial_box mass="6" x="0.2" y="0.18" z="0.12" >
+        <xacro:inertial_box mass="6" x="0.2" y="0.30" z="0.12" >
             <origin xyz="0.0 0.0 0.0" rpy="0.0 0.0 0.0"/>
         </xacro:inertial_box>
         <collision>
-            <origin xyz="0.0 0.0 0.0" rpy="0.0 0.0 0.0"/>
+            <origin xyz="0.0 0.0 0.02" rpy="0.0 0.0 0.0"/>
                 <geometry>
-                    <box size="0.2 0.36 0.12 "/>
+                    <box size="0.2 0.36 0.14 "/>
                 </geometry>
         </collision>
@@ -37,5 +31,5 @@
                 <box size=".025 .025 .025"/>
             </geometry>
-            <material name="red"/>
+                <material name="red"/>
         </visual>
     </link>

File: models/project_robot/urdf/wheel.xacro (robot description, xacro)
@@ -11,11 +11,4 @@
                 <material name="black"/>
             </visual>
-            <!-- <visual name='wheel_${side}_visual'>
-                <origin xyz="${(sign*0.1)/8} 0 0" rpy="0 ${pi/2} 0"/>
-                <geometry>
-                    <cylinder length="${(0.1)/4}" radius="${0.15/2}"/>
-                </geometry>
-                <material name="black"/>
-            </visual> -->
             <xacro:inertial_cylinder mass="1" length="${(0.1)/4}" radius="${0.15/2}">
                 <origin xyz="${(sign*0.1)/8} 0 0" rpy="0 ${pi/2} 0"/>
@@ -31,6 +24,6 @@
             <origin xyz="${x*sign} ${y} ${z}" rpy="0 0 0"/>
             <axis xyz="1 0 0" />
-            <limit effort="100" velocity="50"/>
-            <joint_properties damping="0.5" friction="0.1"/>
+                <limit effort="100" velocity="50"/>
+                <joint_properties damping="0.5" friction="0.1"/>
             <child link="wheel_${side}"/>
             <parent link="base"/>

Commit message: exam

File: models/project_robot/urdf/robot_model.xacro (robot description, xacro)
@@ -1,5 +1,5 @@
 <?xml version='1.0'?>
 <robot name="project_robot" xmlns:xacro="http://www.ros.org/wiki/xacro" >
-<xacro:property name="pack" value="roscourse_2023_project_scene" />
+<xacro:property name="pack" value="roscourse_2023_project_scene_368201" />
 <xacro:include filename="$(find ${pack})/models/project_robot/urdf/materials.xacro" />
 <xacro:include filename="$(find ${pack})/models/project_robot/urdf/wheel.xacro" />
@@ -9,5 +9,5 @@
     <link name='base'>
         <visual name='base_visual'>
-            <origin xyz="0.033 -0.025 -0.05" rpy=" 0 0 ${-pi/2}"/>
+            <origin xyz="0.033 -0.025 -0.06" rpy=" 0 0 ${-pi/2}"/>
             <geometry>
                 <mesh filename="$(find ${pack})/models/Subaru_Impreza.stl" scale="0.08 0.1 0.11"/>
@@ -16,10 +16,10 @@
         </visual>
         <xacro:inertial_box mass="6" x="0.2" y="0.30" z="0.12" >
-            <origin xyz="0.0 0.0 0.0" rpy="0.0 0.0 0.0"/>
+            <origin xyz="0.0 0.0 -0.02" rpy="0.0 0.0 0.0"/>
         </xacro:inertial_box>
         <collision>
-            <origin xyz="0.0 0.0 0.02" rpy="0.0 0.0 0.0"/>
+            <origin xyz="0.0 0.0 0.005" rpy="0.0 0.0 0.0"/>
                 <geometry>
-                    <box size="0.2 0.36 0.14 "/>
+                    <box size="0.2 0.3 0.14 "/>
                 </geometry>
         </collision>

File: models/project_robot/urdf/wheel.xacro (robot description, xacro)
@@ -2,5 +2,5 @@
 <robot xmlns:xacro="http://www.ros.org/wiki/xacro">
     <xacro:macro name="wheel" params="side x y z sign sign2">
-        <xacro:property name="pack" value="roscourse_2023_project_scene" />
+        <xacro:property name="pack" value="roscourse_2023_project_scene_368201" />
         <link name='wheel_${side}'>
             <visual name='wheel_${side}_visual'>
@@ -17,5 +17,5 @@
                <origin xyz="${(sign*0.1)/8} 0 0" rpy="0 ${pi/2} 0"/>
                 <geometry>
-                    <cylinder length="${(0.1)/4}" radius="${0.15/2}"/>
+                    <cylinder length="${(0.1)/4}" radius="${0.17/2}"/>
                 </geometry>
             </collision>

Commit message: пгл

File: models/project_robot/urdf/robot_model.xacro (robot description, xacro)
@@ -19,5 +19,5 @@
         </xacro:inertial_box>
         <collision>
-            <origin xyz="0.0 0.0 0.005" rpy="0.0 0.0 0.0"/>
+            <origin xyz="0.0 0.0 0.01" rpy="0.0 0.0 0.0"/>
                 <geometry>
                     <box size="0.2 0.3 0.14 "/>

File: models/project_robot/urdf/wheel.xacro (robot description, xacro)
@@ -11,5 +11,5 @@
                 <material name="black"/>
             </visual>
-            <xacro:inertial_cylinder mass="1" length="${(0.1)/4}" radius="${0.15/2}">
+            <xacro:inertial_cylinder mass="1" length="${(0.1)/4}" radius="${0.17/2}">
                 <origin xyz="${(sign*0.1)/8} 0 0" rpy="0 ${pi/2} 0"/>
             </xacro:inertial_cylinder>
@@ -17,5 +17,5 @@
                <origin xyz="${(sign*0.1)/8} 0 0" rpy="0 ${pi/2} 0"/>
                 <geometry>
-                    <cylinder length="${(0.1)/4}" radius="${0.15/2}"/>
+                    <cylinder length="${(0.1)/4}" radius="${0.17/2}"/>
                 </geometry>
             </collision>
